File: 電路設計/kicad/incense_p0.kicad_sch (KiCad schematic)
At the start: 9 parts, among them J1 K型熱電偶, J2 12V 2A 變壓器, M1 5015 渦輪風扇 12V 0.2A, U2 SCD41 CO2 (0x62) - I2C1 埠, U3 GY-SHT31-D (0x44) - I2C2 埠, U5 MAX6675 熱電偶介面, U6 D4184 MOSFET 模組

Commit message: NVMe 遷移+比賽現場模式落地:SD 卡除役、致動段三處真 bug 修復
- Pi5:SD 卡讀取層退化除役,aroma01 角色移植到 NVMe(Pironman 5);
  冷開機全自動就緒實測通過,唯一手動步驟=R4 電源鍵(內建電池設計)
- 比賽模式:手機熱點無條件最優先(60s 巡檢跳槽)、熱點上雲演練通過、
  看門狗 v2(查資料流非只查裝置)、udev 固定名 /dev/r4
- 韌體:ioWrite() 補多工器通道切換(原碼致動指令會落到錯誤通道)、
  PCF8574 改 I2C3 獨佔埠(CH_PCF=2,免分接線)★待重燒錄★
- KiCad:理香致動段 08-07 起從未成功生成——補齊 PCF/K1/M2/LED1 佈線、
  修 U6 撞名(PCF→U7)、修 K1/M2 超出圖紙;13 元件 24 網路驗證全過
- 接線圖 rev F:致動段、聯鎖 150/130、12V 3A、R4 電源鍵與 /dev/r4 註記
- 部署紀錄:三個附錄(NVMe 遷移、現場演練、冷開機測試)
- 交接任務_筆電接手.md:外地接手 SOP 與 PCF 存廢待決事項

Co-Authored-By: Claude Fable 5 <noreply@anthropic.com>
Parts:
- added K1: 電磁鐵 ×4（理香，脈衝驅動）, symbol incense:Solenoid-Array
- added LED1: 罩內 LED 側光 12V, symbol incense:Hood-LED
- added M2: 超音波霧化模組 12V（冷霧，無明火）, symbol incense:Mist-Ultrasonic
- added U7: I2C 8路 MOSFET 驅動板, symbol incense:PCF8574-MOSFET
- J2: value 12V 2A 變壓器 -> 12V 3A 變壓器
Connections:
- net +12V: now also U7.5 (VIN+ 12V)
- net +5V: now also U7.1 (VCC 5V)
- net GND: now also LED1.2 (GND), M2.2 (GND), U7.2 (GND)
- new net HOODLED: LED1.1 (HOODLED), U7.11 (OUT6 罩內LED)
- new net I2C3_SCL: A1.14 (I2C3 SCL), U7.4 (SCL)
- new net I2C3_SDA: A1.13 (I2C3 SDA), U7.3 (SDA)
- new net MAG1: K1.1 (MAG1), U7.6 (OUT1 電磁鐵1)
- new net MAG2: K1.2 (MAG2), U7.7 (OUT2 電磁鐵2)
- new net MAG3: K1.3 (MAG3), U7.8 (OUT3 電磁鐵3)
- new net MAG4: K1.4 (MAG4), U7.9 (OUT4 電磁鐵4)
- new net MIST: M2.1 (MIST), U7.10 (OUT5 霧化)
